File: PCB/pcb-reflow-hot-plate/pcb-reflow-hot-plate.kicad_pcb (KiCad board)
At the start: 2 copper layers, 80 x 60 mm, 67 parts, among them J1 USB-C, J2 AC In, J3 OLED Display, J4 Heater, J5 Thermocouple, K1 G3MB202PDC12, Q1 HX2301A, Q2 HX2301A, SW1 Boot, SW5 Reset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

Commit message: PCB Rev 1.2
Parts:
- added C9: 100n, Capacitor_SMD:C_0402_1005Metric, F.Cu at (132.6, 93.1)
- added D6: WS2812B, LED_SMD:LED_WS2812B_PLCC4_5.0x5.0mm_P3.2mm, F.Cu at (137.0, 94.2)
- added F1: Fuse, Fuse:Fuse_Littelfuse_395Series, F.Cu at (123.0, 55.5)
- added J6: JST-SH, Connector_JST:JST_SH_SM04B-SRSS-TB_1x04-1MP_P1.00mm_Horizontal, F.Cu at (137.0, 102.8)
- BZ1: footprint Buzzer_Beeper:Buzzer_12x9.5RM7.6 -> pcb-reflow-hot-plate:CMI-9653S-SMT-TR
- Q1, Q2: value HX2301A -> BSS138
- moved R5 12.1 mm to (157.9, 63.2)
- moved D5 9.04 mm to (155.1, 64.2), turned to 180 degrees
- moved BZ1 4.36 mm to (170.5, 94.7), turned to 90 degrees
- moved H5 1.48 mm to (148.8, 71.7)
- moved H8 1.48 mm to (125.2, 71.7)
- moved H6 1.43 mm to (125.2, 95.2)
- moved H7 1.43 mm to (148.8, 95.2)
- moved G*** 1.30 mm to (110.5, 54.5)
- moved G*** 1.25 mm to (105.6, 68.1)
- moved G*** 1.10 mm to (121.1, 102.2)
- moved J3 0.80 mm to (133.2, 70.7)
- moved K1 0.60 mm to (137.0, 65.4)
Connections:
- net Net-(U5-GPIO8) renamed LED
- J2 pad 2: AC_L -> Net-(J2-Pin_2)
Routing:
- net +3V3: track 143.9 -> 177.3 mm, vias 1 -> 4
- net SDA: track 31.9 -> 60.2 mm, vias 2 -> 4
- net LED: track 1.62 -> 29.2 mm
- net SCL: track 36.0 -> 63.3 mm, vias 2 -> 4
- net GND: track 90.6 -> 116.5 mm, vias 43 -> 46
- net Net-(J2-Pin_2): track 0.00 -> 13.2 mm
- net AC_L: track 69.9 -> 57.8 mm
- net SSR: track 24.0 -> 29.3 mm
- net Net-(D3-A): track 79.8 -> 77.9 mm
- net Net-(BZ1-+): track 15.1 -> 16.1 mm
- net Net-(D5-K): track 1.57 -> 2.32 mm
- net +5V: track 36.5 -> 35.9 mm
- net AC_N: track 49.3 -> 49.9 mm
Other:
- board text added: "AC 110V ~2A"
- board text added: "Rev 1.2"
- board text added: "SCL SDA 3V3 GND"
- board text removed: "AC Input 110V"
- board text removed: "Heat"
- board text removed: "Mount using M2 standoffs"
- board text removed: "Rev 1.1"

Commit message: pcb rev 1.3
Parts:
- removed J6: JST-SH, Connector_JST:JST_SH_SM04B-SRSS-TB_1x04-1MP_P1.00mm_Horizontal
- moved C9 7.40 mm to (132.6, 100.5)
- moved D6 7.40 mm to (137.0, 101.6)
- moved G*** 0.61 mm to (121.0, 102.8)
- turned J4 to 80 degrees
- turned J5 to -80 degrees
Connections:
- J5 pad 1: Net-(J5-Pin_1) -> GND
- U3 pad 2: Net-(J5-Pin_1) -> GND
Routing:
- net SDA: track 60.2 -> 31.9 mm, vias 4 -> 2
- net SCL: track 63.3 -> 36.1 mm, vias 4 -> 2
- net +3V3: track 177.3 -> 166.1 mm, vias 4 -> 2
- net Net-(J5-Pin_1): track 6.59 -> 0.00 mm
- net LED: track 29.2 -> 34.9 mm
- net GND: track 116.5 -> 118.1 mm, vias 46 -> 45
- net Net-(J5-Pin_2): track 6.59 -> 6.00 mm
Other:
- board text added: "Rev 1.3"
- board text removed: "Rev 1.2"
- board text removed: "SCL SDA 3V3 GND"
