File: PCB/pcb-reflow-hot-plate/pcb-reflow-hot-plate.kicad_sch (KiCad schematic)
At the start: 63 parts, among them J1 USB-C, J2 AC In, J3 OLED Display, J4 Heater, J5 Thermocouple, K1 G3MB202PDC12, Q1 HX2301A, Q2 HX2301A, SW1 Boot, SW5 Reset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

Commit message: PCB Rev 1.2
Parts:
- added C9: 100n, Capacitor_SMD:C_0402_1005Metric, symbol Device:C
- added D6: WS2812B, LED_SMD:LED_WS2812B_PLCC4_5.0x5.0mm_P3.2mm, symbol LED:WS2812B
- added F1: Fuse, Fuse:Fuse_Littelfuse_395Series, symbol Device:Fuse
- added J6: JST-SH, Connector_JST:JST_SH_SM04B-SRSS-TB_1x04-1MP_P1.00mm_Horizontal, symbol Connector_Generic:Conn_01x04
- BZ1: footprint Buzzer_Beeper:Buzzer_12x9.5RM7.6 -> pcb-reflow-hot-plate:CMI-9653S-SMT-TR
- Q1, Q2: value HX2301A -> BSS138; LCSC Part Number C296298 -> C2874697; Manufacturer HX -> JSMSEMI; Part Number HX2301A -> BSS138
Connections:
- net +3V3: now also C9.1, D6.1 (VDD), J6.3 (Pin_3)
- net AC_L: now also F1.2; no longer J2.2 (Pin_2)
- net GND: now also C9.2, D6.3 (VSS), J6.4 (Pin_4)
- net SCL: now also J6.1 (Pin_1)
- net SDA: now also J6.2 (Pin_2)
- net LED: now reaches R13.2, U5.22 (GPIO8)
- net LED: now also D6.4 (DIN)
- new net: F1.1, J2.2 (Pin_2)
Other:
- note added: "RGB LED"
- moved on the sheet: BZ1, C3, C4, C5, C6, C8, D1, D2, D3, D4, D5, H1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

Commit message: pcb rev 1.3
Parts:
- removed J6: JST-SH, Connector_JST:JST_SH_SM04B-SRSS-TB_1x04-1MP_P1.00mm_Horizontal, symbol Connector_Generic:Conn_01x04
Connections:
- net GND: now also J5.1 (Pin_1), U3.2 (T-)
